File: MSPBOIADV.sch (EAGLE design)
At the start: 23 parts, among them IC1 W25Q32JVDAIQ, U1 MSP430G2553IRHB32T, U2 MSP430G2553IRHB32T

Commit message: Add files via upload
Fixed board, added 28 pin MSP, and through hole flash chip
Parts:
- removed U1, U2: MSP430G2553IRHB32T, ELEC327:MSP430G2553IRHB32T
- added U$3: MSP430G2XX3TSSOP, ELEC327:MSP430G2XX3TSSOP
- added U$5: USETHIS, TI_MSP430_v16:USETHIS
Connections:
- removed net CLOCK: IC1.CLK
- removed net DATA_FLASH: IC1.DO, U2.P2.0/TA1.0
- removed net DATA_INPUT: IC1.DI, U2.P1.1/TA0.0/UCA0RXD/UCA0SOMI/A1/CA1, U2.P2.2/TA1.1
- removed net DATA_OUTPUT: U2.P1.2/TA0.1/UCA0TXD/UCA0SIMO/A2/CA2
- removed net DB7: U$2.P$15, U2.P2.4/TA1.2
- new net N$11: U$5.11
- new net N$12: U$5.12
- new net N$13: U$5.13
- new net N$14: U$5.14
- new net O_CLK: IC1.SCK, U$5.6
- new net O_SIMO: IC1.SI, U$5.4
- new net O_SOMI: IC1.SO, U$5.3
- net A0: now also U$5.18
- net BTN1: now also U$5.20; no longer U2.P3.6/TA0.2
- net BTN2: now also U$3.13; no longer U2.P3.5/TA0.1
- net C86: now also U$5.21; no longer U2.P3.7/TA1CLK/CAOUT
- net CHP_SLCT: now also U$3.8; no longer U1.P3.0/TA0.2, U2.P1.4/SMCLK/UCB0STE/UCA0CLK/VREF+/VEREF+/A4/CA4/TCK
- net CS1: now also U$5.9; no longer U2.P3.0/TA0.2
- net CS_FLASH: now also IC1.CS, U$5.8; no longer IC1./CS, U2.P3.1/TA1.0
- net E/RD: now also U$5.16; no longer U2.P2.3/TA1.0
- net GND: now also U$3.20, U$5.28; no longer U1.DVSS, U2.DVSS
- net HOLD: now also IC1.HOLD, U$5.10, U$5.27; no longer IC1./HOLD, U2.P3.2/TA1.1
- net P/S: now also U$5.26; no longer U2.P2.5/TA1.2
- net RES: now also U$5.15; no longer U2.P3.3/TA1.2
- net RST: now also U$3.16; no longer U1.!RST/NMI/SBWTDIO
- net RST2: now also U$5.24; no longer U2.!RST/NMI/SBWTDIO
- net RW/WR: now also U$5.17; no longer U2.P3.4/TA0.0
- net S_CLK_SPI: now also U$3.7, U$5.7; no longer U1.P1.5/TA0.0/UCB0CLK/UCA0STE/A5/CA5/TMS, U2.P1.5/TA0.0/UCB0CLK/UCA0STE/A5/CA5/TMS
- net S_SIMO: now also U$2.P$15, U$3.15, U$5.23; no longer U1.P1.7/CAOUT/UCB0SIMO/UCB0SDA/A7/CA7/TDO/TDI, U2.P1.7/CAOUT/UCB0SIMO/UCB0SDA/A7/CA7/TDO/TDI
- net S_SOMI: now also U$3.14, U$5.22; no longer U1.P1.6/TA0.1/UCB0SOMI/UCB0SCL/A6/CA6/TDI/TCLK, U2.P1.6/TA0.1/UCB0SOMI/UCB0SCL/A6/CA6/TDI/TCLK
- net TEST: now also U$3.17; no longer U1.TEST/SBWTCK
- net TEST2: now also U$5.25; no longer U2.TEST/SBWTCK
- net VCC: now also U$3.1, U$5.1; no longer U1.DVCC, U2.DVCC
- net WRITE_PROTC: now also IC1.WP, U$5.19; no longer IC1./WP, U2.P2.1/TA1.1
- net X: now also U$5.2; no longer U2.P1.0/TA0CLK/ACLK/A0/CA0
- net Y: now also U$5.5; no longer U2.P1.3/ADC10CLK/CAOUT/VREF-/VEREF-/A3/CA3
